Commit message: base release

File: src/vehicle/vehicle_sim/urdf/bike.urdf (robot description, URDF)
Before this commit: robot prius, 5 links, 4 joints
Links:
- link front_left_wheel: geometry collision sphere radius=0.31265; visual mesh filename=package://vehicle_sim/meshes/wheel.obj scale=0.01 0.01 0.01
- link rear_left_wheel: geometry collision sphere radius=0.31265; visual mesh filename=package://vehicle_sim/meshes/wheel.obj scale=0.01 0.01 0.01
- link steering_wheel: geometry visual mesh filename=package://vehicle_sim/meshes/steering_wheel.obj scale=0.01 0.01 0.01
